File: fan-controller_research/fan-controller_research.sch (KiCad schematic (older format))
At the start: 0 parts

Commit message: Frequency characteristics: Signal transformer.
Changed lines of the file:
@@
 $Descr A4 11693 8268
 encoding utf-8
-Sheet 1 2
+Sheet 1 3
 Title ""
 Date ""
@@
 F1 "test_frequecy-transfer_tl071_01.sch" 60
 $EndSheet
+$Sheet
+S 850  1700 1000 600
+U 5906D7CA
+F0 "test_frequecy-transfer_ T60403-K5032-X102_01" 60
+F1 "test_frequecy-transfer_ T60403-K5032-X102_01.sch" 60
+$EndSheet
 $EndSCHEMATC
