File: fan-controller_research/fan-controller_research.sch (KiCad schematic (older format))
At the start: 0 parts

Commit message: Communication system
Changed lines of the file:
@@
 LIBS:contrib
 LIBS:valves
+LIBS:74xgxx
+LIBS:ac-dc
+LIBS:actel
+LIBS:allegro
+LIBS:Altera
+LIBS:analog_devices
+LIBS:battery_management
+LIBS:bbd
+LIBS:bosch
+LIBS:brooktre
+LIBS:cmos_ieee
+LIBS:dc-dc
+LIBS:diode
+LIBS:elec-unifil
+LIBS:ESD_Protection
+LIBS:ftdi
+LIBS:gennum
+LIBS:graphic
+LIBS:hc11
+LIBS:infineon
+LIBS:intersil
+LIBS:ir
+LIBS:Lattice
+LIBS:leds
+LIBS:LEM
+LIBS:logo
+LIBS:maxim
+LIBS:mechanical
+LIBS:microchip_dspic33dsc
+LIBS:microchip_pic10mcu
+LIBS:microchip_pic12mcu
+LIBS:microchip_pic16mcu
+LIBS:microchip_pic18mcu
+LIBS:microchip_pic24mcu
+LIBS:microchip_pic32mcu
+LIBS:modules
+LIBS:motor_drivers
+LIBS:motors
+LIBS:msp430
+LIBS:nordicsemi
+LIBS:nxp
+LIBS:nxp_armmcu
+LIBS:onsemi
+LIBS:Oscillators
+LIBS:powerint
+LIBS:Power_Management
+LIBS:pspice
+LIBS:references
+LIBS:relays
+LIBS:rfcom
+LIBS:RFSolutions
+LIBS:sensors
+LIBS:silabs
+LIBS:stm8
+LIBS:stm32
+LIBS:supertex
+LIBS:switches
+LIBS:transf
+LIBS:triac_thyristor
+LIBS:ttl_ieee
+LIBS:video
+LIBS:wiznet
+LIBS:Worldsemi
+LIBS:Xicor
+LIBS:zetex
+LIBS:Zilog
 LIBS:fan-controller_research-cache
 EELAYER 25 0
 EELAYER END
-$Descr A4 11693 8268
+$Descr A3 16535 11693
 encoding utf-8
-Sheet 1 4
-Title ""
+Sheet 1 12
+Title "Research master sheet"
 Date ""
 Rev ""
@@
 $EndDescr
 $Sheet
-S 850  850  1000 600
+S 550  600  1000 600
 U 59031321
 F0 "test_frequecy-transfer_tl071_01" 60
@@
 $EndSheet
 $Sheet
-S 3100 850  1000 600
+S 3100 600  1000 600
 U 5906D7CA
 F0 "test_frequecy-transfer_ T60403-K5032-X102_01" 60
@@
 $EndSheet
 $Sheet
-S 5900 850  1000 550
+S 550  1400 1000 550
 U 59071FE0
 F0 "test_frequecy-transfer_filter_15000_01" 60
 F1 "test_frequecy-transfer_filter_15000_01.sch" 60
 $EndSheet
+$Sheet
+S 3100 1400 1000 550
+U 5910AF65
+F0 "test_frequecy-transfer_filter_20000_01" 60
+F1 "test_frequecy-transfer_filter_20000_01.sch" 60
+$EndSheet
+$Sheet
+S 6100 1400 1000 550
+U 59120F8E
+F0 "test_frequecy-transfer_filter_25000_01" 60
+F1 "test_frequecy-transfer_filter_25000_01.sch" 60
+$EndSheet
+$Sheet
+S 550  2900 1000 550
+U 59331C59
+F0 "test_50kHz_power-amp" 60
+F1 "test_50kHz_power-amp.sch" 60
+$EndSheet
+$Sheet
+S 542  3658 1008 542
+U 59437D3A
+F0 "test_jfet_01" 60
+F1 "test_jfet_01.sch" 60
+$EndSheet
+$Sheet
+S 3100 3650 1000 550
+U 59439CCC
+F0 "test_wien-bridge-osc_fet-agc_15000-20000-25000" 60
+F1 "test_wien-bridge-osc_fet-agc.sch" 60
+$EndSheet
+$Sheet
+S 6100 4400 1000 550
+U 594BA696
+F0 "test_analog-sig-switch_4066" 60
+F1 "test_analog-sig-switch_4066.sch" 60
+$EndSheet
+$Sheet
+S 550  4400 1000 550
+U 594FC379
+F0 "test_analog-sig-switch_4066_single" 60
+F1 "test_analog-sig-switch_4066_single.sch" 60
+$EndSheet
+$Sheet
+S 3100 4400 1000 550
+U 5950A101
+F0 "test_analog-switch_4066_chopper" 60
+F1 "test_analog-switch_4066_chopper.sch" 60
+$EndSheet
+$Sheet
+S 6100 2100 1050 600
+U 5955993D
+F0 "test_frequency-transfer_filter_passive_25000_01" 39
+F1 "test_frequency-transfer_filter_passive_25000_01.sch" 39
+$EndSheet
 $EndSCHEMATC
