File: fan-controller_research/test_frequecy-transfer_tl071_01.sch (KiCad schematic (older format))
At the start: 9 parts, among them U201 TL071

Commit message: Frequency characteristics: Signal transformer.
Other:
- note added: "0 Hz ... 50 kHz\n\nMarker is \nat 30 kHz."
- note removed: "0 Hz ... 50 kHz\n\nMarker is at 30 kHz."
Changed lines of the file:
@@
 $Descr A4 11693 8268
 encoding utf-8
-Sheet 2 2
+Sheet 2 3
 Title "Frequency transfer, TL071"
 Date "2017-04-28"
@@
 	1    0    0    -1
 $EndComp
-Text Notes 5900 1100 0    79   ~ 0
+Text Notes 6650 750  0    79   ~ 0
 Spectrum analyzer output
-Text Notes 9550 1250 0    79   ~ 0
+Text Notes 10100 900  0    79   ~ 0
 0Hz ... 5MHz
-Text Notes 9550 4150 0    79   ~ 0
-0 Hz ... 50 kHz\n\nMarker is at 30 kHz.
+Text Notes 10100 3950 0    79   ~ 0
+0 Hz ... 50 kHz\n\nMarker is \nat 30 kHz.
 $Bitmap
-Pos 7600 2450
+Pos 8350 2100
 Scale 1.000000
 Data
 89 50 4E 47 0D 0A 1A 0A 00 00 00 0D 49 48 44 52 00 00 04 00 00 00 03 07 08 02 00 00 00 28 DD B2
-E2 00 00 00 03 73 42 49 54 08 08 08 DB E1 4F E0 00 00 00 09 70 48 59 73 00 00 0E C3 00 00 0E C3
-01 C7 6F A8 64 00 00 20 00 49 44 41 54 78 9C EC BD 7D 7F EB B8 AA 28 0C C8 4E DA AE 99 7D 7E E7
+E2 00 00 00 03 73 42 49 54 08 08 08 DB E1 4F E0 00 00 00 09 70 48 59 73 00 00 0E 74 00 00 0E 74
+01 6B 24 B3 D6 00 00 20 00 49 44 41 54 78 9C EC BD 7D 7F EB B8 AA 28 0C C8 4E DA AE 99 7D 7E E7
 FB 7F C8 F3 DC 7B E7 4C 9B C4 12 CF 1F 48 18 4B C2 B1 D3 A4 ED 9A 09 7B 6D 8F AB C8 08 BD 21 40
 08 E1 7F DE 5E 01 00 00 10 51 9F 00 C0 CC D0 03 2F 3D C6 D8 4D 57 E4 57 31 5B 32 F6 00 ED C2 A3
@@
 $EndBitmap
 $Bitmap
-Pos 7600 5150
+Pos 8350 4800
 Scale 1.000000
 Data
 89 50 4E 47 0D 0A 1A 0A 00 00 00 0D 49 48 44 52 00 00 04 00 00 00 03 29 08 02 00 00 00 15 7B D6
-A4 00 00 00 03 73 42 49 54 08 08 08 DB E1 4F E0 00 00 00 09 70 48 59 73 00 00 0E C3 00 00 0E C3
-01 C7 6F A8 64 00 00 20 00 49 44 41 54 78 9C EC BD DB B2 E4 B8 CE 26 F6 01 D4 AA EA 7D 98 F0 1F
+A4 00 00 00 03 73 42 49 54 08 08 08 DB E1 4F E0 00 00 00 09 70 48 59 73 00 00 0E 74 00 00 0E 74
+01 6B 24 B3 D6 00 00 20 00 49 44 41 54 78 9C EC BD DB B2 E4 B8 CE 26 F6 01 D4 AA EA 7D 98 F0 1F
 F6 D8 11 E3 08 DF F9 FD 1F CF B3 A7 2B 45 F8 02 24 04 81 07 49 99 CA B5 AA BA 0B 5D 5B 5B 8B 49
 81 20 08 82 00 78 A2 FF F7 FF FE 2F 00 22 22 22 00 88 88 88 00 FC F9 E7 9F 00 34 C5 9E 9A 13 3D
@@
 $EndComp
 Wire Wire Line
-	3200 3900 3200 4100
-Wire Wire Line
-	3200 4100 3200 4750
+	3200 3900 3200 4750
 Wire Wire Line
 	3000 3700 2850 3700
@@
 	2850 4500 4100 4500
 Wire Wire Line
-	1550 4300 1550 4550
-Wire Wire Line
-	1550 4550 1550 4750
+	1550 4300 1550 4750
 Wire Wire Line
-	3200 3300 3200 3050
-Wire Wire Line
-	3200 3050 3200 2600
+	3200 2600 3200 3300
 Wire Wire Line
 	4700 4350 4700 4750
 Wire Wire Line
-	2150 3500 2500 3500
-Wire Wire Line
-	2500 3500 3000 3500
+	2150 3500 3000 3500
 Wire Wire Line
 	1850 3500 1550 3500
@@
 	1550 3500 1550 4100
 Wire Wire Line
-	3600 3600 4100 3600
-Wire Wire Line
-	4100 3600 4250 3600
+	3600 3600 4250 3600
 Wire Wire Line
 	4100 4500 4100 3600
@@
 Connection ~ 1550 4550
 Wire Notes Line
-	5400 700  5400 7500
-Wire Wire Line
-	1250 950  1250 1050
-Wire Wire Line
-	1250 1050 1250 1150
-Wire Wire Line
-	1250 1450 1250 1600
+	6200 700  6200 7500
 Wire Wire Line
-	1250 1600 1250 1700
+	1250 950  1250 1150
 Wire Wire Line
-	1250 2000 1250 2100
+	1250 1450 1250 1700
 Wire Wire Line
-	1250 2100 1250 2200
+	1250 2000 1250 2200
 Wire Wire Line
 	1750 1650 1750 1600
