File: fan-controller_modules/comms/oscillator/osc_25k/osc_25k.kicad_pcb (KiCad board)
At the start: 2 copper layers, 177.8 x 71.1 mm, 63 parts, among them J101 PWR, J102 UNMUTE, J103 SIG_OUT, Q201 2N3819, Q301 BC546, Q302 BC546, Q303 BC546, Q304 BC556, U201 TL061, U202 TL061, U301 4066, U302 TL061

Commit message: Comms, Oscillator, 25k -> Finalized
Parts:
- moved C204 44.8 mm to (160.4, 109.1)
- moved C304 12.1 mm to (219.6, 108.5), turned to 270 degrees
- moved D303 11.2 mm to (180.7, 84.9), turned to 270 degrees
- moved C306 8.93 mm to (204.9, 108.1), turned to 90 degrees
- moved R305 6.86 mm to (183.4, 82.9), turned to 180 degrees
- moved C305 6.35 mm to (223.9, 106.6)
- moved R315 6.04 mm to (193.4, 112.7)
- moved R303 2.41 mm to (186.3, 91.1), turned to 180 degrees
- moved R304 2.29 mm to (195.6, 91.1), turned to 180 degrees
- moved U302 1.40 mm to (212.1, 107.8)
- moved R201 1.27 mm to (85.6, 86.6), turned to 0 degrees
- moved C201 0.63 mm to (88.1, 88.8)
- moved R311 0.36 mm to (193.0, 101.6), turned to 0 degrees
- moved R313 0.36 mm to (189.2, 101.6), turned to 0 degrees
- moved R309 0.36 mm to (186.7, 101.6), turned to 0 degrees
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Routing:
- net /_VEE: track 188.7 -> 268.3 mm, vias 4 -> 5
- net /_VCC: track 155.5 -> 233.7 mm, vias 4 -> 5
- net GND: track 26.0 -> 100.0 mm, vias 6 -> 16
- net /subcirc_switch/_VCC_2: track 0.00 -> 71.8 mm, vias 0 -> 3
- net Net-(C204-Pad1): track 9.48 -> 65.0 mm
- net /subcirc_switch/_VEE_2: track 0.00 -> 48.2 mm, vias 0 -> 1
- net /subcirc_switch/SIG_IN: track 0.00 -> 39.9 mm, vias 0 -> 2
- net /subcirc_switch/SIG_OUT: track 0.00 -> 36.4 mm
- net (no net): track 0.00 -> 30.5 mm, vias 0 -> 11
- net Net-(R314-Pad2): track 0.00 -> 26.7 mm, vias 0 -> 2
- net Net-(R315-Pad2): track 0.00 -> 25.2 mm
- net Net-(R312-Pad2): track 0.00 -> 21.7 mm, vias 0 -> 2
- net Net-(Q303-Pad1): track 0.00 -> 19.4 mm
- net Net-(D303-Pad1): track 0.00 -> 17.1 mm
- net Net-(Q302-Pad1): track 0.00 -> 15.6 mm
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- added copper zone on B.Cu, net GND
Other:
- rule trace_min: 0.01 -> 0.2
- board text added: "+15V"
- board text added: "-15V"
- board text added: "AGC"
- board text added: "FEEDBK"
- board text added: "GND"
- board text added: "HOT"
- board text added: "OUT"
- board text added: "Oscillator, 25kHz, AGC stabilized, switchable Evaluation board Ver 1.0"
- board text added: "PWR"
- board text added: "SIG"
- board text added: "UNMUTE"
