File: schematics/controller/controller.sch (KiCad schematic (older format))
At the start: 57 parts, among them J1001 Screw_Terminal_01x03, J1002 Screw_Terminal_01x03, J1003 Periphery, J1004 Conn_01x02_Male, J1005 Conn_01x04_Male, J1006 Conn_01x04_Male, J1007 FRONTPANEL, U1001 Module: surgeprot.mains.275.5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, U1002 Bourns 2026-07-C2LF, U1003 Bourns 2026-07-C2LF, U1004 Bourns 2026-07-C2LF

Commit message: Upgraded KiCad to v.5 and made plans compatible Implementing PCB
Parts:
- removed D1001, D1003, D1004, D1006, D1007, D1009: 1.5KE33CA, Diodes_THT:D_DO-201AD_P12.70mm_Horizontal, symbol D_TVS
- D1002, D1005, D1008, D1010, D1011, D1012, D1013, D1014, D1015, D1016, D1017, D1018: symbol D_TVS -> Device:D_TVS
- F1001, F1002, F1003, F1004, F1005, F1006, F1007, F1008, F1009, F1010, F1011, F1012: symbol Fuse -> Device:Fuse
- J1001, J1002: symbol Screw_Terminal_01x03 -> conn:Screw_Terminal_01x03
- J1003: symbol Screw_Terminal_01x12 -> conn:Screw_Terminal_01x12
- J1004: symbol Conn_01x02_Male -> conn:Conn_01x02_Male
- J1005, J1006: symbol Conn_01x04_Male -> conn:Conn_01x04_Male
- J1007: symbol Conn_01x05_Male -> conn:Conn_01x05_Male
- MK1001, MK1002, MK1003, MK1004, MK1005, MK1006, MK1007, MK1008, MK1009, MK1010: symbol Mounting_Hole_PAD -> mechanical:Mounting_Hole_PAD
- R1001, R1002, R1003, R1004, R1005, R1006: symbol R -> device:R
- U1001: symbol line-protector -> fan-controller_parts:line-protector
- U1002, U1003, U1004: symbol GDT-3 -> ESD_Protection:GDT-3
