File: schematics/controller/controller.kicad_pcb (KiCad board)
At the start: 2 copper layers, 355 parts, among them J1001 Screw_Terminal_01x03, J1002 Screw_Terminal_01x03, J1003 Periphery, J1004 Conn_01x02_Male, J1005 Conn_01x04_Male, J1006 Conn_01x04_Male, J1007 FRONTPANEL, K2001 TE RT424024 (24VDC@1.44kOhm, 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, Q10001 BC546C, Q10002 BC546C, Q10003 BC546C, Q10004 BC556, Q12001 BC556, Q12002 BC556, Q12003 BC546C, Q12004 BC546C, Q12005 BC546C, Q12006 BC546C, Q12007 BC546C, Q12008 BC546C, Q14001 BC546C, Q14002 BC546C, Q14003 BC546C, Q14004 BC546C, Q14005 BC546C, Q15001 BC546C, Q2001 BC556, Q2002 BC546C, Q2003 BD243C, Q6001 2N3819, Q7001 BC546C, Q7002 BC546C, Q7003 BC546C, Q7004 BC556, Q9001 2N3819, T13001 Transformer_2P_1S, U10001 4066, U10002 TL061, U1001 Module: surgeprot.mains.275.5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, U1002 Bourns 2026-07-C2LF, U1003 Bourns 2026-07-C2LF, U1004 Bourns 2026-07-C2LF, U11001 OP282, U11002 OP282, U12001 TL061, U12002 TL061, U12003 TL061, U13001 OP282, U3001 L7805, U3002 L7815, U3003 L7915, U6001 TL061, U6002 TL061, U7001 4066, U7002 TL061, U9001 TL061, U9002 TL061

Commit message: Upgraded KiCad to v.5 and made plans compatible Implementing PCB
Parts:
- removed D1001, D1003, D1004, D1006, D1007, D1009: 1.5KE33CA, Diodes_THT:D_DO-201AD_P12.70mm_Horizontal
- moved F1007 319.6 mm to (244.9, 94.0), turned to 180 degrees
- moved R1001 314.9 mm to (277.5, 93.3), turned to 180 degrees
- moved R1005 305.4 mm to (277.5, 43.8), turned to 180 degrees
- moved F1008 304.3 mm to (244.9, 83.8), turned to 180 degrees
- moved R1002 302.6 mm to (277.5, 84.5), turned to 180 degrees
- moved D1010 296.9 mm to (304.8, 94.0), turned to 180 degrees
- moved R1003 288.1 mm to (277.5, 73.0), turned to 180 degrees
- moved D1013 286.1 mm to (304.8, 74.3), turned to 180 degrees
- moved D1018 285.7 mm to (304.8, 54.0), turned to 180 degrees
- moved D1015 284.4 mm to (304.8, 64.1), turned to 180 degrees
- moved D1012 284.2 mm to (304.8, 83.8), turned to 180 degrees
- moved F1009 283.1 mm to (244.9, 73.7), turned to 180 degrees
- moved F1005 282.8 mm to (171.6, 83.8)
- moved R1004 280.7 mm to (277.5, 64.8), turned to 180 degrees
- moved F1010 277.4 mm to (244.9, 63.5), turned to 180 degrees
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Connections:
- net /comms/sub_assy/comms/barrier/OSC_15K_SIG_OUT_10BAUD_SDA renamed /comms/comms/barrier/OSC_15K_SIG_OUT_10BAUD_SDA
- net /comms/sub_assy/comms/barrier/OSC_25K_SIG_OUT_10BAUD_SCL renamed /comms/comms/barrier/OSC_25K_SIG_OUT_10BAUD_SCL
- net /comms/sub_assy/comms/detector_15k/IN renamed /comms/comms/detector_15k/IN
- net /comms/sub_assy/comms/filter_15k/IN renamed /comms/comms/filter_15k/IN
- net /comms/sub_assy/comms/osc_15k/sub_assy/comms/osc_15k/osc/OUT renamed /comms/comms/osc_15k/osc_15k/osc/OUT
- net /comms/sub_assy/comms/osc_25k/sub_assy/comms/osc_25k/osc/OUT renamed /comms/comms/osc_25k/osc_25k/osc/OUT
Other:
- board text added: "+18V"
- board text added: "0V"
- board text added: "GND"
- board text added: "X"
- board text added: "Y"

Commit message: Implementing PCB.
Parts:
- F2001: footprint Wire_Connections_Bridges:WireConnection_2.50mmDrill_LargePad -> Fuse_Holders_and_Fuses:Fuseholder5x20_horiz_open_Schurter_0031_8201
- moved J1006 356.6 mm to (45.7, 198.1), turned to 90 degrees
- moved J1005 322.2 mm to (45.7, 152.4), turned to 90 degrees
- moved K2001 280.1 mm to (85.1, 96.5), turned to 90 degrees
- moved F3006 268.7 mm to (57.1, 194.3)
- moved F3005 266.2 mm to (57.1, 204.5)
- moved F3001 238.0 mm to (57.1, 157.5)
- moved F2001 234.9 mm to (78.7, 54.6)
- moved F3007 222.9 mm to (57.1, 184.2)
- moved F3008 221.9 mm to (57.1, 174.0)
- moved F3002 214.5 mm to (57.1, 147.3)
- moved J1004 213.8 mm to (45.7, 96.5), turned to 90 degrees
- moved F3003 213.2 mm to (57.1, 137.2)
- moved MK1001 191.4 mm to (25.4, 25.4)
- moved F3004 181.4 mm to (57.1, 127.0)
- moved J1001 174.0 mm to (55.9, 35.6), turned to 180 degrees
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Other:
- board text added: "E"
- board text added: "FAN"
- board text added: "L"
- board text added: "MAINS"
- board text added: "N"
